Commit message: Fix SLAM map freeze: enable RPLIDAR angle_compensate, load mapper_params_async.yaml, set A2M8 range limits; add joystick config; hardware-verified wheel mapping

File: description/lidar.xacro (robot description, xacro)
@@ -4,5 +4,5 @@
         <parent link="chassis"/>
         <child link="laser_frame"/>
-        <origin xyz="0.122 0 0.212" rpy="0 0 0"/>
+        <origin xyz="0.17 0 0.212" rpy="0 0 3.14159"/>
     </joint>
     <link name="laser_frame">

File: description/ros2_control.xacro (robot description, xacro)
@@ -11,5 +11,5 @@
                 <param name="baud_rate">57600</param>
                 <param name="timeout">1000</param>
-                <param name="enc_counts_per_rev">3450</param>
+                <param name="enc_counts_per_rev">510</param>
             </hardware>
             <joint name="left_wheel_joint">
